Commit message: arm板卡端重新编译gazbeo classic；模型文件加载改成相对路径

File: src/gazebo_quadbot/robot_scene/xacro/go2_leg.xacro (robot description, xacro)
@@ -42,5 +42,5 @@
                 </xacro:if>
                 <geometry>
-                    <mesh filename="file://$(find go2_description)/meshes/hip.dae" scale="1 1 1"/>
+                    <mesh filename="package://go2_description/meshes/hip.dae" scale="1 1 1"/>
                 </geometry>
                 <!-- <material name="orange"/> -->
@@ -74,8 +74,8 @@
                 <geometry>
                     <xacro:if value="${mirror_dae == True}">
-                        <mesh filename="file://$(find go2_description)/meshes/thigh.dae" scale="1 1 1"/>
+                        <mesh filename="package://go2_description/meshes/thigh.dae" scale="1 1 1"/>
                     </xacro:if>
                     <xacro:if value="${mirror_dae == False}">
-                        <mesh filename="file://$(find go2_description)/meshes/thigh_mirror.dae" scale="1 1 1"/>
+                        <mesh filename="package://go2_description/meshes/thigh_mirror.dae" scale="1 1 1"/>
                     </xacro:if>
                 </geometry>
@@ -109,5 +109,5 @@
                 <origin rpy="0 0 0" xyz="0 0 0"/>
                 <geometry>
-                    <mesh filename="file://$(find go2_description)/meshes/calf.dae" scale="1 1 1"/>
+                    <mesh filename="package://go2_description/meshes/calf.dae" scale="1 1 1"/>
                 </geometry>
                 <!-- <material name="orange"/> -->

File: src/gazebo_quadbot/robot_scene/xacro/go2_robot_VLP.xacro (robot description, xacro)
@@ -37,5 +37,5 @@
             <origin rpy="0 0 0" xyz="0 0 0"/>
             <geometry>
-                <mesh filename="file://$(find go2_description)/meshes/trunk.dae" scale="1 1 1"/>
+                <mesh filename="package://go2_description/meshes/trunk.dae" scale="1 1 1"/>
             </geometry>
             <!-- <material name="orange"/> -->

File: src/gazebo_quadbot/robot_scene/xacro/go2w_description.urdf.xacro (robot description, xacro)
@@ -3,5 +3,5 @@
   <!-- Gloabal parameters -->
   <xacro:include filename="$(find robot_scene)/xacro/go2w_const.xacro"/>
-  <xacro:property name="mesh_prefix" value="file://$(find go2w_description)/meshes" />
+  <xacro:property name="mesh_prefix" value="package://go2w_description/meshes" />
   <xacro:macro name="leg" params="prefix front left">
     <xacro:if value="${(front == True)}">

File: src/gazebo_quadbot/robot_scene/xacro/mid360.xacro (robot description, xacro)
@@ -27,6 +27,5 @@
         <origin xyz="0 0 -0.045" rpy="0 0 0"/>
         <geometry>
-          <mesh filename="file://$(find mid360_simulation)/meshes/livox_frame.STL"/>
-          <!-- <mesh filename="$(find mid360_simulation)/meshes/livox_frame.STL"/> -->
+          <mesh filename="package://mid360_simulation/meshes/livox_frame.STL"/>
         </geometry>
         <material name="livox_dark_grey">
@@ -37,6 +36,5 @@
         <origin xyz="-0.011 -0.02329 -0.005" rpy="0 0 0"/>
         <geometry>
-          <mesh filename="file://$(find mid360_simulation)/meshes/livox_frame.STL"/>
-          <!-- <mesh filename="$(find mid360_simulation)/meshes/livox_frame.STL"/> -->
+          <mesh filename="package://mid360_simulation/meshes/livox_frame.STL"/>
         </geometry>
       </collision>
@@ -83,4 +81,7 @@
         <pose>0 0 0 0 0 0</pose>
         <visualize>true</visualize>
+        <!-- Gazebo 默认 always_on=false：传感器不主动更新，
+             必须显式打开，否则 RayPlugin 的 OnNewLaserScans 永不回调 -->
+        <always_on>true</always_on>
         <update_rate>${update_rate}</update_rate>
         <plugin name="${name}_plugin" filename="libmid360_plugin.so">
