Commit message: 延时加载机器狗模型；删除重复启动

File: src/gazebo_quadbot/robot_scene/xacro/mid360.xacro (robot description, xacro)
@@ -27,5 +27,6 @@
         <origin xyz="0 0 -0.045" rpy="0 0 0"/>
         <geometry>
-          <mesh filename="$(find mid360_simulation)/meshes/livox_frame.STL"/>
+          <mesh filename="file://$(find mid360_simulation)/meshes/livox_frame.STL"/>
+          <!-- <mesh filename="$(find mid360_simulation)/meshes/livox_frame.STL"/> -->
         </geometry>
         <material name="livox_dark_grey">
@@ -36,5 +37,6 @@
         <origin xyz="-0.011 -0.02329 -0.005" rpy="0 0 0"/>
         <geometry>
-          <mesh filename="$(find mid360_simulation)/meshes/livox_frame.STL"/>
+          <mesh filename="file://$(find mid360_simulation)/meshes/livox_frame.STL"/>
+          <!-- <mesh filename="$(find mid360_simulation)/meshes/livox_frame.STL"/> -->
         </geometry>
       </collision>

Commit message: 修改go2w无法正常启动的bug

File: src/gazebo_quadbot/robot_scene/xacro/mid360.xacro (robot description, xacro)
@@ -33,10 +33,7 @@
         </material>
       </visual>
-      <collision>
-        <origin xyz="-0.011 -0.02329 -0.005" rpy="0 0 0"/>
-        <geometry>
-          <mesh filename="package://mid360_simulation/meshes/livox_frame.STL"/>
-        </geometry>
-      </collision>
+      <!-- 不设碰撞体：雷达 link 若带 trimesh 碰撞，always_on 的 ray 传感器
+           首次扫描即触发 ODE ray-vs-trimesh 段错误（gzserver exit -11）；
+           传感器 link 无碰撞体是常规做法，radar 固定在 trunk/base_link 上不影响运动 -->
     </link>
     <joint name="${name}_joint" type="fixed">
